File: pico-ice40-1k/hw-picow-1k/prj_kicad/picow-1k.kicad_pcb (KiCad board)
At the start: 2 copper layers, 100 x 72 mm, 133 parts, among them P1 CONN_RJ45-L, P2 CONN_VGA, P3 CONN_DC-2.0, P4 CONN_20X2, Q901 BC846, SW1 SW_PUSH, SW2 SW_PUSH, SW3 SW_PUSH, SW4 SW_PUSH, SW900 SW_PUSH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

Commit message: = UPD: board routing - ready for verification
Parts:
- added agilack-11.5: 450px, agilack-11.5, F.Cu at (130.4, 101.3)
- added ohw_logo: VAL**, ohw-logo, F.Cu at (148.1, 99.8)
Routing:
- net GND: track 506.4 -> 987.7 mm, vias 103 -> 145
- net +3.3V: track 317.1 -> 645.1 mm, vias 17 -> 32
- net +1.2V: track 29.7 -> 105.1 mm
- net BUT3: track 0.00 -> 58.8 mm, vias 0 -> 2
- net PLD_CS: track 0.00 -> 56.2 mm, vias 0 -> 2
- net PLD_MISO: track 0.00 -> 55.8 mm, vias 0 -> 4
- net PLD_SCK: track 0.00 -> 54.6 mm, vias 0 -> 2
- net PLD_MOSI: track 0.00 -> 51.4 mm, vias 0 -> 2
- net BUT4: track 0.00 -> 50.0 mm
- net BUT2: track 0.00 -> 49.3 mm
- net PLD_RST: track 0.00 -> 47.7 mm, vias 0 -> 2
- net PLD_DONE: track 0.00 -> 46.7 mm, vias 0 -> 2
- net LCD_DC: track 0.00 -> 44.8 mm, vias 0 -> 2
- net LCD_CS: track 0.00 -> 42.8 mm, vias 0 -> 2
- net BUT1: track 0.00 -> 40.6 mm
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Other:
- board text added: "Agilack 2015 CC-by-SA"
- board text added: "eCow-Logic ice40-1k"
