File: pico-ice40-1k/hw-picow-1k/board-rev-0.2/prj_kicad/picow-1k-display.sch (KiCad schematic (older format))
At the start: 45 parts, among them P2 CONN_VGA, U101 AS6C4008, U102 TLV61220, U103 74AHC157

Commit message: = UPD: Improve schema, change IOs/extension connector (HE10 pins), fix display
Parts:
- added C108: C, symbol C
- added C109: 47uF, symbol C
- added L103: INDUCTOR, symbol INDUCTOR
Connections:
- net labels added: LCD_RST
- wire segments 173 -> 179
Changed lines of the file:
@@
 $EndComp
 $Comp
-L GND #PWR065
+L GND #PWR067
 U 1 1 5641EE9D
 P 10100 2550
-F 0 "#PWR065" H 10100 2550 30  0001 C CNN
+F 0 "#PWR067" H 10100 2550 30  0001 C CNN
 F 1 "GND" H 10100 2480 30  0001 C CNN
 F 2 "" H 10100 2550 60  0000 C CNN
@@
 Connection ~ 10100 2450
 $Comp
-L GND #PWR066
+L GND #PWR068
 U 1 1 5641EEB0
 P 10300 2550
-F 0 "#PWR066" H 10300 2550 30  0001 C CNN
+F 0 "#PWR068" H 10300 2550 30  0001 C CNN
 F 1 "GND" H 10300 2480 30  0001 C CNN
 F 2 "" H 10300 2550 60  0000 C CNN
@@
 $EndComp
 $Comp
-L GND #PWR067
+L GND #PWR069
 U 1 1 5641EF2E
 P 5950 1600
-F 0 "#PWR067" H 5950 1600 30  0001 C CNN
+F 0 "#PWR069" H 5950 1600 30  0001 C CNN
 F 1 "GND" H 5950 1530 30  0001 C CNN
 F 2 "" H 5950 1600 60  0000 C CNN
@@
 $EndComp
 $Comp
-L GND #PWR068
+L GND #PWR070
 U 1 1 5641F716
 P 5950 2400
-F 0 "#PWR068" H 5950 2400 30  0001 C CNN
+F 0 "#PWR070" H 5950 2400 30  0001 C CNN
 F 1 "GND" H 5950 2330 30  0001 C CNN
 F 2 "" H 5950 2400 60  0000 C CNN
@@
 $EndComp
 $Comp
-L GND #PWR069
+L GND #PWR071
 U 1 1 5641FAB3
 P 5950 3200
-F 0 "#PWR069" H 5950 3200 30  0001 C CNN
+F 0 "#PWR071" H 5950 3200 30  0001 C CNN
 F 1 "GND" H 5950 3130 30  0001 C CNN
 F 2 "" H 5950 3200 60  0000 C CNN
@@
 $EndComp
 $Comp
-L GND #PWR070
+L GND #PWR072
 U 1 1 5643393F
 P 5550 4700
-F 0 "#PWR070" H 5550 4700 30  0001 C CNN
+F 0 "#PWR072" H 5550 4700 30  0001 C CNN
 F 1 "GND" H 5550 4630 30  0001 C CNN
 F 2 "" H 5550 4700 60  0000 C CNN
@@
 Wire Wire Line
 	1950 6400 1950 6600
-Wire Wire Line
-	1650 6600 2750 6600
 $Comp
 L TLV61220 U102
@@
 	2750 6400 2650 6400
 Connection ~ 1950 6600
-Wire Wire Line
-	1650 6500 1650 6600
 Connection ~ 1750 6600
 $Comp
-L +3.3V #PWR071
+L +3.3V #PWR073
 U 1 1 56433BF0
-P 1650 6500
-F 0 "#PWR071" H 1650 6460 30  0001 C CNN
-F 1 "+3.3V" H 1650 6610 30  0000 C CNN
-F 2 "" H 1650 6500 60  0000 C CNN
-F 3 "" H 1650 6500 60  0000 C CNN
-	1    1650 6500
-	1    0    0    -1
-$EndComp
-$Comp
-L GND #PWR072
+P 750 6400
+F 0 "#PWR073" H 750 6360 30  0001 C CNN
+F 1 "+3.3V" H 750 6510 30  0000 C CNN
+F 2 "" H 750 6400 60  0000 C CNN
+F 3 "" H 750 6400 60  0000 C CNN
+	1    750  6400
+	1    0    0    -1
+$EndComp
+$Comp
+L GND #PWR074
 U 1 1 56433BFF
 P 1750 7200
-F 0 "#PWR072" H 1750 7200 30  0001 C CNN
+F 0 "#PWR074" H 1750 7200 30  0001 C CNN
 F 1 "GND" H 1750 7130 30  0001 C CNN
 F 2 "" H 1750 7200 60  0000 C CNN
@@
 	1750 7200 1750 7100
 $Comp
-L GND #PWR073
+L GND #PWR075
 U 1 1 56434117
 P 4200 5600
-F 0 "#PWR073" H 4200 5600 30  0001 C CNN
+F 0 "#PWR075" H 4200 5600 30  0001 C CNN
 F 1 "GND" H 4200 5530 30  0001 C CNN
 F 2 "" H 4200 5600 60  0000 C CNN
@@
 	4200 5600 4200 5550
 $Comp
-L GND #PWR074
+L GND #PWR076
 U 1 1 56434410
 P 3150 7100
-F 0 "#PWR074" H 3150 7100 30  0001 C CNN
+F 0 "#PWR076" H 3150 7100 30  0001 C CNN
 F 1 "GND" H 3150 7030 30  0001 C CNN
 F 2 "" H 3150 7100 60  0000 C CNN
@@
 $EndComp
 Wire Wire Line
-	3550 6400 4500 6400
+	3550 6400 4800 6400
 Wire Wire Line
 	3900 6400 3900 6450
@@
 $EndComp
 $Comp
-L GND #PWR075
+L GND #PWR077
 U 1 1 56433C25
 P 3900 7600
-F 0 "#PWR075" H 3900 7600 30  0001 C CNN
+F 0 "#PWR077" H 3900 7600 30  0001 C CNN
 F 1 "GND" H 3900 7530 30  0001 C CNN
 F 2 "" H 3900 7600 60  0000 C CNN
@@
 $EndComp
 $Comp
-L GND #PWR076
+L GND #PWR078
 U 1 1 56433BD5
 P 4300 7000
-F 0 "#PWR076" H 4300 7000 30  0001 C CNN
+F 0 "#PWR078" H 4300 7000 30  0001 C CNN
 F 1 "GND" H 4300 6930 30  0001 C CNN
 F 2 "" H 4300 7000 60  0000 C CNN
@@
 	4300 6400 4300 6500
 Connection ~ 3900 6400
-Wire Wire Line
-	4500 6400 4500 6300
 Connection ~ 4300 6400
 $Comp
-L +VDISP #PWR077
+L +VDISP #PWR079
 U 1 1 56434025
-P 4500 6300
-F 0 "#PWR077" H 4500 6260 30  0001 C CNN
-F 1 "+VDISP" H 4500 6410 30  0000 C CNN
-F 2 "" H 4500 6300 60  0000 C CNN
-F 3 "" H 4500 6300 60  0000 C CNN
-	1    4500 6300
-	1    0    0    -1
-$EndComp
-$Comp
-L +3.3V #PWR078
+P 4800 6300
+F 0 "#PWR079" H 4800 6260 30  0001 C CNN
+F 1 "+VDISP" H 4800 6410 30  0000 C CNN
+F 2 "" H 4800 6300 60  0000 C CNN
+F 3 "" H 4800 6300 60  0000 C CNN
+	1    4800 6300
+	1    0    0    -1
+$EndComp
+$Comp
+L +3.3V #PWR080
 U 1 1 56433D02
 P 4200 4150
-F 0 "#PWR078" H 4200 4110 30  0001 C CNN
+F 0 "#PWR080" H 4200 4110 30  0001 C CNN
 F 1 "+3.3V" H 4200 4260 30  0000 C CNN
 F 2 "" H 4200 4150 60  0000 C CNN
@@
 $EndComp
 $Comp
-L +VDISP #PWR079
+L +VDISP #PWR081
 U 1 1 56433D11
 P 4000 4150
-F 0 "#PWR079" H 4000 4110 30  0001 C CNN
+F 0 "#PWR081" H 4000 4110 30  0001 C CNN
 F 1 "+VDISP" H 4000 4260 30  0000 C CNN
 F 2 "" H 4000 4150 60  0000 C CNN
@@
 $EndComp
 $Comp
-L GND #PWR080
+L GND #PWR082
 U 1 1 564340F9
 P 5050 5900
-F 0 "#PWR080" H 5050 5900 30  0001 C CNN
+F 0 "#PWR082" H 5050 5900 30  0001 C CNN
 F 1 "GND" H 5050 5830 30  0001 C CNN
 F 2 "" H 5050 5900 60  0000 C CNN
@@
 	3550 5900 3550 5850
 $Comp
-L GND #PWR081
+L GND #PWR083
 U 1 1 56433EC3
 P 3550 5900
-F 0 "#PWR081" H 3550 5900 30  0001 C CNN
+F 0 "#PWR083" H 3550 5900 30  0001 C CNN
 F 1 "GND" H 3550 5830 30  0001 C CNN
 F 2 "" H 3550 5900 60  0000 C CNN
@@
 	2850 5050 3650 5050
 $Comp
-L GND #PWR082
+L GND #PWR084
 U 1 1 56449189
 P 1700 5700
-F 0 "#PWR082" H 1700 5700 30  0001 C CNN
+F 0 "#PWR084" H 1700 5700 30  0001 C CNN
 F 1 "GND" H 1700 5630 30  0001 C CNN
 F 2 "" H 1700 5700 60  0000 C CNN
@@
 	1700 3800 1700 3850
 $Comp
-L +3.3V #PWR083
+L +3.3V #PWR085
 U 1 1 564492B3
 P 1700 3800
-F 0 "#PWR083" H 1700 3760 30  0001 C CNN
+F 0 "#PWR085" H 1700 3760 30  0001 C CNN
 F 1 "+3.3V" H 1700 3910 30  0000 C CNN
 F 2 "" H 1700 3800 60  0000 C CNN
@@
 	1250 5100 1350 5100
 $Comp
-L +3.3V #PWR084
+L +3.3V #PWR086
 U 1 1 5644A9DA
 P 2200 900
-F 0 "#PWR084" H 2200 860 30  0001 C CNN
+F 0 "#PWR086" H 2200 860 30  0001 C CNN
 F 1 "+3.3V" H 2200 1010 30  0000 C CNN
 F 2 "" H 2200 900 60  0000 C CNN
@@
 	2200 3300 2200 3250
 $Comp
-L GND #PWR085
+L GND #PWR087
 U 1 1 5644AB1C
 P 2200 3300
-F 0 "#PWR085" H 2200 3300 30  0001 C CNN
+F 0 "#PWR087" H 2200 3300 30  0001 C CNN
 F 1 "GND" H 2200 3230 30  0001 C CNN
 F 2 "" H 2200 3300 60  0000 C CNN
@@
 	1250 4800 1350 4800
 $Comp
-L GND #PWR086
+L GND #PWR088
 U 1 1 5644BEDF
 P 9350 5950
-F 0 "#PWR086" H 9350 5950 30  0001 C CNN
+F 0 "#PWR088" H 9350 5950 30  0001 C CNN
 F 1 "GND" H 9350 5880 30  0001 C CNN
 F 2 "" H 9350 5950 60  0000 C CNN
@@
 $EndComp
 $Comp
-L +3.3V #PWR087
+L +3.3V #PWR089
 U 1 1 564B7733
 P 3450 2300
-F 0 "#PWR087" H 3450 2260 30  0001 C CNN
+F 0 "#PWR089" H 3450 2260 30  0001 C CNN
 F 1 "+3.3V" H 3450 2410 30  0000 C CNN
 F 2 "" H 3450 2300 60  0000 C CNN
@@
 $EndComp
 $Comp
-L GND #PWR088
+L GND #PWR090
 U 1 1 564B7742
 P 3450 2800
-F 0 "#PWR088" H 3450 2800 30  0001 C CNN
+F 0 "#PWR090" H 3450 2800 30  0001 C CNN
 F 1 "GND" H 3450 2730 30  0001 C CNN
 F 2 "" H 3450 2800 60  0000 C CNN
@@
 	3450 2350 3450 2300
 $Comp
-L +VIN #PWR089
+L +VIN #PWR091
 U 1 1 564C5496
 P 10100 900
-F 0 "#PWR089" H 10100 860 30  0001 C CNN
+F 0 "#PWR091" H 10100 860 30  0001 C CNN
 F 1 "+VIN" H 10100 1010 30  0000 C CNN
 F 2 "" H 10100 900 60  0000 C CNN
@@
 Wire Wire Line
 	10100 900  10100 950
+$Comp
+L INDUCTOR L103
+U 1 1 56903D38
+P 1350 6600
+F 0 "L103" V 1300 6600 40  0000 C CNN
+F 1 "INDUCTOR" V 1450 6600 40  0000 C CNN
+F 2 "" H 1350 6600 60  0000 C CNN
+F 3 "" H 1350 6600 60  0000 C CNN
+	1    1350 6600
+	0    -1   -1   0
+$EndComp
+Wire Wire Line
+	1650 6600 2750 6600
+$Comp
+L C C108
+U 1 1 56904052
+P 950 6900
+F 0 "C108" H 1000 7000 50  0000 L CNN
+F 1 "C" H 1000 6800 50  0000 L CNN
+F 2 "" H 950 6900 60  0000 C CNN
+F 3 "" H 950 6900 60  0000 C CNN
+	1    950  6900
+	1    0    0    -1
+$EndComp
+$Comp
+L GND #PWR092
+U 1 1 56904061
+P 950 7200
+F 0 "#PWR092" H 950 7200 30  0001 C CNN
+F 1 "GND" H 950 7130 30  0001 C CNN
+F 2 "" H 950 7200 60  0000 C CNN
+F 3 "" H 950 7200 60  0000 C CNN
+	1    950  7200
+	1    0    0    -1
+$EndComp
+Wire Wire Line
+	950  7200 950  7100
+Wire Wire Line
+	950  6700 950  6600
+Wire Wire Line
+	750  6600 1050 6600
+Wire Wire Line
+	750  6400 750  6600
+Connection ~ 950  6600
+$Comp
+L C C109
+U 1 1 5690FAC9
+P 4700 6700
+F 0 "C109" H 4750 6800 50  0000 L CNN
+F 1 "47uF" H 4750 6600 50  0000 L CNN
+F 2 "" H 4700 6700 60  0000 C CNN
+F 3 "" H 4700 6700 60  0000 C CNN
+F 4 "Murata" H 4700 6700 60  0001 C CNN "Manufacturer"
+F 5 "GRM21BR61E226ME44L" H 4700 6700 60  0001 C CNN "Manuf Ref"
+	1    4700 6700
+	1    0    0    -1
+$EndComp
+Wire Wire Line
+	4800 6400 4800 6300
+Wire Wire Line
+	4700 6500 4700 6400
+Connection ~ 4700 6400
+Wire Wire Line
+	4700 7000 4700 6900
+$Comp
+L GND #PWR093
+U 1 1 5690FD3B
+P 4700 7000
+F 0 "#PWR093" H 4700 7000 30  0001 C CNN
+F 1 "GND" H 4700 6930 30  0001 C CNN
+F 2 "" H 4700 7000 60  0000 C CNN
+F 3 "" H 4700 7000 60  0000 C CNN
+	1    4700 7000
+	1    0    0    -1
+$EndComp
+Text GLabel 3550 4550 0    45   Input ~ 0
+LCD_RST
+Wire Wire Line
+	3550 4550 3650 4550
 $EndSCHEMATC
