File: pico-ice40-1k/hw-picow-1k/board-rev-0.2/prj_kicad/picow-1k-io.sch (KiCad schematic (older format))
At the start: 13 parts, among them P4 CONN_20X2, SW1 SW_PUSH, SW2 SW_PUSH, SW3 SW_PUSH, SW4 SW_PUSH

Commit message: = UPD: Improve schema, change IOs/extension connector (HE10 pins), fix display
Parts:
- removed P4: CONN_20X2, symbol CONN_20X2
- added P4, P5: CONN_12, symbol CONN_12
- added P6: CONN_2, symbol CONN_2
- added TP151, TP152: CONN_1, symbol CONN_1
Connections:
- net labels added: +VIN
- wire segments 73 -> 58
