File: pico-ice40-1k/hardware/prj_kicad/picow-1k-display.sch (KiCad schematic (older format))
At the start: 48 parts, among them P2 CONN_VGA, U101 AS6C4008, U102 TLV61220, U103 74AHC157

Commit message: = UPD: Update hardware for rev 0.2.1 board (mainly bugfix)
Parts:
- C109: value 47uF -> 22uF
- L101: value 4,7uH -> 10uH; Manuf Ref (none) -> TYS4012100M-10; Manufacturer (none) -> Laird Technologies
- R121, R123: value R -> 120
- R122: value R -> 60
Changed lines of the file:
@@
 $EndComp
 $Comp
-L GND #PWR067
+L GND #PWR068
 U 1 1 5641EE9D
 P 10100 2550
-F 0 "#PWR067" H 10100 2550 30  0001 C CNN
+F 0 "#PWR068" H 10100 2550 30  0001 C CNN
 F 1 "GND" H 10100 2480 30  0001 C CNN
 F 2 "" H 10100 2550 60  0000 C CNN
@@
 Connection ~ 10100 2450
 $Comp
-L GND #PWR068
+L GND #PWR069
 U 1 1 5641EEB0
 P 10300 2550
-F 0 "#PWR068" H 10300 2550 30  0001 C CNN
+F 0 "#PWR069" H 10300 2550 30  0001 C CNN
 F 1 "GND" H 10300 2480 30  0001 C CNN
 F 2 "" H 10300 2550 60  0000 C CNN
@@
 $EndComp
 $Comp
-L GND #PWR069
+L GND #PWR070
 U 1 1 5641EF2E
 P 5950 1600
-F 0 "#PWR069" H 5950 1600 30  0001 C CNN
+F 0 "#PWR070" H 5950 1600 30  0001 C CNN
 F 1 "GND" H 5950 1530 30  0001 C CNN
 F 2 "" H 5950 1600 60  0000 C CNN
@@
 $EndComp
 $Comp
-L GND #PWR070
+L GND #PWR071
 U 1 1 5641F716
 P 5950 2400
-F 0 "#PWR070" H 5950 2400 30  0001 C CNN
+F 0 "#PWR071" H 5950 2400 30  0001 C CNN
 F 1 "GND" H 5950 2330 30  0001 C CNN
 F 2 "" H 5950 2400 60  0000 C CNN
@@
 P 6950 2650
 F 0 "R123" V 7050 2650 50  0000 C CNN
-F 1 "R" V 6950 2650 50  0000 C CNN
+F 1 "120" V 6950 2650 50  0000 C CNN
 F 2 "" H 6950 2650 60  0000 C CNN
 F 3 "" H 6950 2650 60  0000 C CNN
@@
 P 6250 2900
 F 0 "R121" V 6350 2900 50  0000 C CNN
-F 1 "R" V 6250 2900 50  0000 C CNN
+F 1 "120" V 6250 2900 50  0000 C CNN
 F 2 "" H 6250 2900 60  0000 C CNN
 F 3 "" H 6250 2900 60  0000 C CNN
@@
 P 6950 3150
 F 0 "R122" V 7050 3150 50  0000 C CNN
-F 1 "R" V 6950 3150 50  0000 C CNN
+F 1 "60" V 6950 3150 50  0000 C CNN
 F 2 "" H 6950 3150 60  0000 C CNN
 F 3 "" H 6950 3150 60  0000 C CNN
@@
 $EndComp
 $Comp
-L GND #PWR071
+L GND #PWR072
 U 1 1 5641FAB3
 P 5950 3200
-F 0 "#PWR071" H 5950 3200 30  0001 C CNN
+F 0 "#PWR072" H 5950 3200 30  0001 C CNN
 F 1 "GND" H 5950 3130 30  0001 C CNN
 F 2 "" H 5950 3200 60  0000 C CNN
@@
 $EndComp
 $Comp
-L GND #PWR072
+L GND #PWR073
 U 1 1 5643393F
 P 5550 4700
-F 0 "#PWR072" H 5550 4700 30  0001 C CNN
+F 0 "#PWR073" H 5550 4700 30  0001 C CNN
 F 1 "GND" H 5550 4630 30  0001 C CNN
 F 2 "" H 5550 4700 60  0000 C CNN
@@
 P 2350 6400
 F 0 "L101" V 2475 6400 60  0000 C CNN
-F 1 "4,7uH" V 2300 6400 45  0000 C CNN
+F 1 "10uH" V 2300 6400 45  0000 C CNN
 F 2 "" H 2350 6400 60  0000 C CNN
 F 3 "" H 2350 6400 60  0000 C CNN
+F 4 "Laird Technologies" V 2350 6400 60  0001 C CNN "Manufacturer"
+F 5 "TYS4012100M-10" V 2350 6400 60  0001 C CNN "Manuf Ref"
 	1    2350 6400
 	0    -1   -1   0
@@
 Connection ~ 1750 6600
 $Comp
-L +3.3V #PWR073
+L +3.3V #PWR074
 U 1 1 56433BF0
 P 750 6400
-F 0 "#PWR073" H 750 6360 30  0001 C CNN
+F 0 "#PWR074" H 750 6360 30  0001 C CNN
 F 1 "+3.3V" H 750 6510 30  0000 C CNN
 F 2 "" H 750 6400 60  0000 C CNN
@@
 $EndComp
 $Comp
-L GND #PWR074
+L GND #PWR075
 U 1 1 56433BFF
 P 1750 7200
-F 0 "#PWR074" H 1750 7200 30  0001 C CNN
+F 0 "#PWR075" H 1750 7200 30  0001 C CNN
 F 1 "GND" H 1750 7130 30  0001 C CNN
 F 2 "" H 1750 7200 60  0000 C CNN
@@
 	1750 7200 1750 7100
 $Comp
-L GND #PWR075
+L GND #PWR076
 U 1 1 56434117
 P 4200 5600
-F 0 "#PWR075" H 4200 5600 30  0001 C CNN
+F 0 "#PWR076" H 4200 5600 30  0001 C CNN
 F 1 "GND" H 4200 5530 30  0001 C CNN
 F 2 "" H 4200 5600 60  0000 C CNN
@@
 	4200 5600 4200 5550
 $Comp
-L GND #PWR076
+L GND #PWR077
 U 1 1 56434410
 P 3150 7100
-F 0 "#PWR076" H 3150 7100 30  0001 C CNN
+F 0 "#PWR077" H 3150 7100 30  0001 C CNN
 F 1 "GND" H 3150 7030 30  0001 C CNN
 F 2 "" H 3150 7100 60  0000 C CNN
@@
 $EndComp
 $Comp
-L GND #PWR077
+L GND #PWR078
 U 1 1 56433C25
 P 3900 7600
-F 0 "#PWR077" H 3900 7600 30  0001 C CNN
+F 0 "#PWR078" H 3900 7600 30  0001 C CNN
 F 1 "GND" H 3900 7530 30  0001 C CNN
 F 2 "" H 3900 7600 60  0000 C CNN
@@
 $EndComp
 $Comp
-L GND #PWR078
+L GND #PWR079
 U 1 1 56433BD5
 P 4300 7000
-F 0 "#PWR078" H 4300 7000 30  0001 C CNN
+F 0 "#PWR079" H 4300 7000 30  0001 C CNN
 F 1 "GND" H 4300 6930 30  0001 C CNN
 F 2 "" H 4300 7000 60  0000 C CNN
@@
 Connection ~ 4300 6400
 $Comp
-L +VDISP #PWR079
+L +VDISP #PWR080
 U 1 1 56434025
 P 4800 6300
-F 0 "#PWR079" H 4800 6260 30  0001 C CNN
+F 0 "#PWR080" H 4800 6260 30  0001 C CNN
 F 1 "+VDISP" H 4800 6410 30  0000 C CNN
 F 2 "" H 4800 6300 60  0000 C CNN
@@
 $EndComp
 $Comp
-L +3.3V #PWR080
+L +3.3V #PWR081
 U 1 1 56433D02
 P 4200 4150
-F 0 "#PWR080" H 4200 4110 30  0001 C CNN
+F 0 "#PWR081" H 4200 4110 30  0001 C CNN
 F 1 "+3.3V" H 4200 4260 30  0000 C CNN
 F 2 "" H 4200 4150 60  0000 C CNN
@@
 $EndComp
 $Comp
-L +VDISP #PWR081
+L +VDISP #PWR082
 U 1 1 56433D11
 P 4000 4150
-F 0 "#PWR081" H 4000 4110 30  0001 C CNN
+F 0 "#PWR082" H 4000 4110 30  0001 C CNN
 F 1 "+VDISP" H 4000 4260 30  0000 C CNN
 F 2 "" H 4000 4150 60  0000 C CNN
@@
 $EndComp
 $Comp
-L GND #PWR082
+L GND #PWR083
 U 1 1 564340F9
 P 5050 5900
-F 0 "#PWR082" H 5050 5900 30  0001 C CNN
+F 0 "#PWR083" H 5050 5900 30  0001 C CNN
 F 1 "GND" H 5050 5830 30  0001 C CNN
 F 2 "" H 5050 5900 60  0000 C CNN
@@
 	3550 5900 3550 5850
 $Comp
-L GND #PWR083
+L GND #PWR084
 U 1 1 56433EC3
 P 3550 5900
-F 0 "#PWR083" H 3550 5900 30  0001 C CNN
+F 0 "#PWR084" H 3550 5900 30  0001 C CNN
 F 1 "GND" H 3550 5830 30  0001 C CNN
 F 2 "" H 3550 5900 60  0000 C CNN
@@
 	2850 5050 3650 5050
 $Comp
-L GND #PWR084
+L GND #PWR085
 U 1 1 56449189
 P 1700 5700
-F 0 "#PWR084" H 1700 5700 30  0001 C CNN
+F 0 "#PWR085" H 1700 5700 30  0001 C CNN
 F 1 "GND" H 1700 5630 30  0001 C CNN
 F 2 "" H 1700 5700 60  0000 C CNN
@@
 	1700 3800 1700 3850
 $Comp
-L +3.3V #PWR085
+L +3.3V #PWR086
 U 1 1 564492B3
 P 1700 3800
-F 0 "#PWR085" H 1700 3760 30  0001 C CNN
+F 0 "#PWR086" H 1700 3760 30  0001 C CNN
 F 1 "+3.3V" H 1700 3910 30  0000 C CNN
 F 2 "" H 1700 3800 60  0000 C CNN
@@
 	1250 5100 1350 5100
 $Comp
-L +3.3V #PWR086
+L +3.3V #PWR087
 U 1 1 5644A9DA
 P 2200 900
-F 0 "#PWR086" H 2200 860 30  0001 C CNN
+F 0 "#PWR087" H 2200 860 30  0001 C CNN
 F 1 "+3.3V" H 2200 1010 30  0000 C CNN
 F 2 "" H 2200 900 60  0000 C CNN
@@
 	2200 3300 2200 3250
 $Comp
-L GND #PWR087
+L GND #PWR088
 U 1 1 5644AB1C
 P 2200 3300
-F 0 "#PWR087" H 2200 3300 30  0001 C CNN
+F 0 "#PWR088" H 2200 3300 30  0001 C CNN
 F 1 "GND" H 2200 3230 30  0001 C CNN
 F 2 "" H 2200 3300 60  0000 C CNN
@@
 	1250 4800 1350 4800
 $Comp
-L GND #PWR088
+L GND #PWR089
 U 1 1 5644BEDF
 P 9350 5950
-F 0 "#PWR088" H 9350 5950 30  0001 C CNN
+F 0 "#PWR089" H 9350 5950 30  0001 C CNN
 F 1 "GND" H 9350 5880 30  0001 C CNN
 F 2 "" H 9350 5950 60  0000 C CNN
@@
 $EndComp
 $Comp
-L +3.3V #PWR089
+L +3.3V #PWR090
 U 1 1 564B7733
 P 3450 2300
-F 0 "#PWR089" H 3450 2260 30  0001 C CNN
+F 0 "#PWR090" H 3450 2260 30  0001 C CNN
 F 1 "+3.3V" H 3450 2410 30  0000 C CNN
 F 2 "" H 3450 2300 60  0000 C CNN
@@
 $EndComp
 $Comp
-L GND #PWR090
+L GND #PWR091
 U 1 1 564B7742
 P 3450 2800
-F 0 "#PWR090" H 3450 2800 30  0001 C CNN
+F 0 "#PWR091" H 3450 2800 30  0001 C CNN
 F 1 "GND" H 3450 2730 30  0001 C CNN
 F 2 "" H 3450 2800 60  0000 C CNN
@@
 	3450 2350 3450 2300
 $Comp
-L +VIN #PWR091
+L +VIN #PWR092
 U 1 1 564C5496
 P 10100 900
-F 0 "#PWR091" H 10100 860 30  0001 C CNN
+F 0 "#PWR092" H 10100 860 30  0001 C CNN
 F 1 "+VIN" H 10100 1010 30  0000 C CNN
 F 2 "" H 10100 900 60  0000 C CNN
@@
 $EndComp
 $Comp
-L GND #PWR092
+L GND #PWR093
 U 1 1 56904061
 P 950 7200
-F 0 "#PWR092" H 950 7200 30  0001 C CNN
+F 0 "#PWR093" H 950 7200 30  0001 C CNN
 F 1 "GND" H 950 7130 30  0001 C CNN
 F 2 "" H 950 7200 60  0000 C CNN
@@
 P 4700 6700
 F 0 "C109" H 4750 6800 50  0000 L CNN
-F 1 "47uF" H 4750 6600 50  0000 L CNN
+F 1 "22uF" H 4750 6600 50  0000 L CNN
 F 2 "" H 4700 6700 60  0000 C CNN
 F 3 "" H 4700 6700 60  0000 C CNN
@@
 	4700 7000 4700 6900
 $Comp
-L GND #PWR093
+L GND #PWR094
 U 1 1 5690FD3B
 P 4700 7000
-F 0 "#PWR093" H 4700 7000 30  0001 C CNN
+F 0 "#PWR094" H 4700 7000 30  0001 C CNN
 F 1 "GND" H 4700 6930 30  0001 C CNN
 F 2 "" H 4700 7000 60  0000 C CNN

Commit message: = UPD: set values and manufacturer ref for components
Parts:
- C101: Manuf Ref (none) -> 0805X106K160CT; Manufacturer (none) -> Walsin
- C105: Manuf Ref (none) -> 0603X225K100CT; Manufacturer (none) -> Walsin
- C106: value C -> 2,2uF; Manuf Ref (none) -> 0603X225K100CT; Manufacturer (none) -> Walsin
- C107: value C -> 100nF; Manuf Ref (none) -> C0603C104K4RACTU; Manufacturer (none) -> Kemet
- L102: value FB100 -> FB120; Manuf Ref (none) -> BLM18TG121TN1D; Manufacturer (none) -> Murata
- L103: value INDUCTOR -> FB120; Manuf Ref (none) -> BLM18TG121TN1D; Manufacturer (none) -> Murata
- R132: Manuf Ref (none) -> CRCW0603560KFKEA; Manufacturer (none) -> Vishay
- R140: Manuf Ref (none) -> CRCW06031K00FKEA; Manufacturer (none) -> Vishay
Changed lines of the file:
@@
 P 5550 4450
 F 0 "C106" H 5600 4550 50  0000 L CNN
-F 1 "C" H 5600 4350 50  0000 L CNN
+F 1 "2,2uF" H 5600 4350 50  0000 L CNN
 F 2 "" H 5550 4450 60  0000 C CNN
 F 3 "" H 5550 4450 60  0000 C CNN
+F 4 "Walsin" H 5550 4450 60  0001 C CNN "Manufacturer"
+F 5 "0603X225K100CT" H 5550 4450 60  0001 C CNN "Manuf Ref"
 	1    5550 4450
 	1    0    0    -1
@@
 F 2 "" H 1750 6900 60  0000 C CNN
 F 3 "" H 1750 6900 60  0000 C CNN
+F 4 "Walsin" H 1750 6900 60  0001 C CNN "Manufacturer"
+F 5 "0805X106K160CT" H 1750 6900 60  0001 C CNN "Manuf Ref"
 	1    1750 6900
 	1    0    0    -1
@@
 F 2 "" H 5050 5600 60  0000 C CNN
 F 3 "" H 5050 5600 60  0000 C CNN
+F 4 "Walsin" H 5050 5600 60  0001 C CNN "Manufacturer"
+F 5 "0603X225K100CT" H 5050 5600 60  0001 C CNN "Manuf Ref"
 	1    5050 5600
 	1    0    0    -1
@@
 F 2 "" H 3550 5600 60  0000 C CNN
 F 3 "" H 3550 5600 60  0000 C CNN
+F 4 "Vishay" V 3550 5600 60  0001 C CNN "Manufacturer"
+F 5 "CRCW0603560KFKEA" V 3550 5600 60  0001 C CNN "Manuf Ref"
 	1    3550 5600
 	1    0    0    -1
@@
 F 2 "" H 8500 3750 60  0000 C CNN
 F 3 "" H 8500 3750 60  0000 C CNN
+F 4 "Vishay" V 8500 3750 60  0001 C CNN "Manufacturer"
+F 5 "CRCW06031K00FKEA" V 8500 3750 60  0001 C CNN "Manuf Ref"
 	1    8500 3750
 	0    -1   -1   0
@@
 P 3450 2550
 F 0 "C107" H 3500 2650 50  0000 L CNN
-F 1 "C" H 3500 2450 50  0000 L CNN
+F 1 "100nF" H 3500 2450 50  0000 L CNN
 F 2 "" H 3450 2550 60  0000 C CNN
 F 3 "" H 3450 2550 60  0000 C CNN
+F 4 "Kemet" H 3450 2550 60  0001 C CNN "Manufacturer"
+F 5 "C0603C104K4RACTU" H 3450 2550 60  0001 C CNN "Manuf Ref"
 	1    3450 2550
 	1    0    0    -1
@@
 P 10100 1250
 F 0 "L102" V 10050 1250 40  0000 C CNN
-F 1 "FB100" V 10200 1250 40  0000 C CNN
+F 1 "FB120" V 10200 1250 40  0000 C CNN
 F 2 "" H 10100 1250 60  0000 C CNN
 F 3 "" H 10100 1250 60  0000 C CNN
+F 4 "Murata" V 10100 1250 60  0001 C CNN "Manufacturer"
+F 5 "BLM18TG121TN1D" V 10100 1250 60  0001 C CNN "Manuf Ref"
 	1    10100 1250
 	1    0    0    -1
@@
 U 1 1 56903D38
 P 1350 6600
-F 0 "L103" V 1300 6600 40  0000 C CNN
-F 1 "INDUCTOR" V 1450 6600 40  0000 C CNN
+F 0 "L103" V 1475 6600 50  0000 C CNN
+F 1 "FB120" V 1300 6600 40  0000 C CNN
 F 2 "" H 1350 6600 60  0000 C CNN
 F 3 "" H 1350 6600 60  0000 C CNN
+F 4 "Murata" V 1350 6600 60  0001 C CNN "Manufacturer"
+F 5 "BLM18TG121TN1D" V 1350 6600 60  0001 C CNN "Manuf Ref"
 	1    1350 6600
 	0    -1   -1   0
