File: pico-ice40-1k/hardware/prj_kicad/picow-1k-net.sch (KiCad schematic (older format))
At the start: 44 parts, among them P1 CONN_RJ45-L, Q901 BC846, SW900 SW_PUSH, SW901 SW_PUSH, T900 TRANSFORMER_1:1, U900 W7500, U901 KSZ8091MNX, U902 M25P16-VME, U903 NCP302, X900 25MHz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

Commit message: = UPD: Update hardware for rev 0.2.1 board (mainly bugfix)
Parts:
- added C921: 10uF, symbol C
- X900: Manuf Ref (none) -> 501JAA25M0000BAF; Manufacturer (none) -> Silicon Labs
Connections:
- wire segments 223 -> 228
- no-connect marks 8 -> 16
Other:
- moved on the sheet: C920, R912, TP903
Changed lines of the file:
@@
 F 2 "" H 1250 3000 60  0000 C CNN
 F 3 "" H 1250 3000 60  0000 C CNN
+F 4 "Silicon Labs" H 1250 3000 60  0001 C CNN "Manufacturer"
+F 5 "501JAA25M0000BAF" H 1250 3000 60  0001 C CNN "Manuf Ref"
 	1    1250 3000
 	1    0    0    -1
@@
 Wire Wire Line
 	7200 4900 7100 4900
-NoConn ~ 5200 4700
-Text GLabel 5100 4600 0    45   Input ~ 0
+Text GLabel 5000 4450 0    45   Input ~ 0
 NET_RST
-Wire Wire Line
-	5100 4600 5200 4600
 $Comp
 L R R907
@@
 L +3.3V #PWR056
 U 1 1 564523FB
-P 5600 6800
-F 0 "#PWR056" H 5600 6760 30  0001 C CNN
-F 1 "+3.3V" H 5600 6910 30  0000 C CNN
-F 2 "" H 5600 6800 60  0000 C CNN
-F 3 "" H 5600 6800 60  0000 C CNN
-	1    5600 6800
+P 5300 6800
+F 0 "#PWR056" H 5300 6760 30  0001 C CNN
+F 1 "+3.3V" H 5300 6910 30  0000 C CNN
+F 2 "" H 5300 6800 60  0000 C CNN
+F 3 "" H 5300 6800 60  0000 C CNN
+	1    5300 6800
 	1    0    0    -1
 $EndComp
@@
 L GND #PWR057
 U 1 1 56452423
-P 5600 7400
-F 0 "#PWR057" H 5600 7400 30  0001 C CNN
-F 1 "GND" H 5600 7330 30  0001 C CNN
-F 2 "" H 5600 7400 60  0000 C CNN
-F 3 "" H 5600 7400 60  0000 C CNN
-	1    5600 7400
-	1    0    0    -1
-$EndComp
-Wire Wire Line
-	5600 7400 5600 7350
-Wire Wire Line
-	5600 7350 6600 7350
-Wire Wire Line
-	5700 7350 5700 7300
-Wire Wire Line
-	5700 6900 5700 6850
-Wire Wire Line
-	5600 6850 6600 6850
-Wire Wire Line
-	5600 6850 5600 6800
+P 5300 7400
+F 0 "#PWR057" H 5300 7400 30  0001 C CNN
+F 1 "GND" H 5300 7330 30  0001 C CNN
+F 2 "" H 5300 7400 60  0000 C CNN
+F 3 "" H 5300 7400 60  0000 C CNN
+	1    5300 7400
+	1    0    0    -1
+$EndComp
+Wire Wire Line
+	5300 7400 5300 7350
+Wire Wire Line
+	5300 7350 6600 7350
+Wire Wire Line
+	5400 7350 5400 7300
+Wire Wire Line
+	5400 6900 5400 6850
+Wire Wire Line
+	5300 6850 6600 6850
+Wire Wire Line
+	5300 6850 5300 6800
 $Comp
 L C C917
@@
 Wire Wire Line
 	6000 6850 6000 6900
-Connection ~ 5700 6850
+Connection ~ 5400 6850
 Wire Wire Line
 	6000 7350 6000 7300
-Connection ~ 5700 7350
+Connection ~ 5400 7350
 $Comp
 L C C918
@@
 L CP C920
 U 1 1 56452EA6
-P 5700 7100
-F 0 "C920" H 5750 7200 50  0000 L CNN
-F 1 "2,2uF" H 5750 7000 50  0000 L CNN
-F 2 "" H 5700 7100 60  0000 C CNN
-F 3 "" H 5700 7100 60  0000 C CNN
-	1    5700 7100
+P 5400 7100
+F 0 "C920" H 5450 7200 50  0000 L CNN
+F 1 "2,2uF" H 5450 7000 50  0000 L CNN
+F 2 "" H 5400 7100 60  0000 C CNN
+F 3 "" H 5400 7100 60  0000 C CNN
+	1    5400 7100
 	1    0    0    -1
 $EndComp
@@
 	10050 3250 10100 3250
 NoConn ~ 1700 5500
-Wire Wire Line
-	5100 4800 5200 4800
 $Comp
 L R R912
 U 1 1 564B0416
-P 4800 4850
-F 0 "R912" V 4900 4850 50  0000 C CNN
-F 1 "10k" V 4805 4850 45  0000 C CNN
-F 2 "" H 4800 4850 60  0000 C CNN
-F 3 "" H 4800 4850 60  0000 C CNN
-	1    4800 4850
+P 4800 4700
+F 0 "R912" V 4700 4700 50  0000 C CNN
+F 1 "10k" V 4805 4700 45  0000 C CNN
+F 2 "" H 4800 4700 60  0000 C CNN
+F 3 "" H 4800 4700 60  0000 C CNN
+	1    4800 4700
 	0    1    1    0
 $EndComp
@@
 L GND #PWR061
 U 1 1 564B0439
-P 4450 4950
-F 0 "#PWR061" H 4450 4950 30  0001 C CNN
-F 1 "GND" H 4450 4880 30  0001 C CNN
-F 2 "" H 4450 4950 60  0000 C CNN
-F 3 "" H 4450 4950 60  0000 C CNN
-	1    4450 4950
-	1    0    0    -1
-$EndComp
-Wire Wire Line
-	4450 4950 4450 4850
-Wire Wire Line
-	4450 4850 4550 4850
-$Comp
-L CONN_1 TP903
-U 1 1 564B0B1F
-P 4650 4750
-F 0 "TP903" H 4730 4750 40  0000 L CNN
-F 1 "CONN_1" H 4650 4805 30  0001 C CNN
-F 2 "" H 4650 4750 60  0000 C CNN
-F 3 "" H 4650 4750 60  0000 C CNN
-	1    4650 4750
-	-1   0    0    1
-$EndComp
-Wire Wire Line
-	4800 4750 5100 4750
-Wire Wire Line
-	5100 4750 5100 4850
-Wire Wire Line
-	5100 4850 5050 4850
-Connection ~ 5100 4800
+P 4450 4800
+F 0 "#PWR061" H 4450 4800 30  0001 C CNN
+F 1 "GND" H 4450 4730 30  0001 C CNN
+F 2 "" H 4450 4800 60  0000 C CNN
+F 3 "" H 4450 4800 60  0000 C CNN
+	1    4450 4800
+	1    0    0    -1
+$EndComp
+Wire Wire Line
+	4450 4800 4450 4700
+Wire Wire Line
+	4450 4700 4550 4700
 Text GLabel 1600 6100 0    45   Output ~ 0
 LCD_EN
@@
 	1    0    0    -1
 $EndComp
+$Comp
+L CONN_1 TP903
+U 1 1 564B0B1F
+P 4800 4800
+F 0 "TP903" H 4880 4800 40  0000 L CNN
+F 1 "CONN_1" H 4800 4855 30  0001 C CNN
+F 2 "" H 4800 4800 60  0000 C CNN
+F 3 "" H 4800 4800 60  0000 C CNN
+	1    4800 4800
+	-1   0    0    1
+$EndComp
+Wire Wire Line
+	5050 4700 5200 4700
+Wire Wire Line
+	4950 4800 5100 4800
+Wire Wire Line
+	5100 4800 5100 4700
+Connection ~ 5100 4700
+$Comp
+L GND #PWR067
+U 1 1 57724F4A
+P 5150 4850
+F 0 "#PWR067" H 5150 4850 30  0001 C CNN
+F 1 "GND" H 5150 4780 30  0001 C CNN
+F 2 "" H 5150 4850 60  0000 C CNN
+F 3 "" H 5150 4850 60  0000 C CNN
+	1    5150 4850
+	1    0    0    -1
+$EndComp
+Wire Wire Line
+	5150 4850 5150 4800
+Wire Wire Line
+	5150 4800 5200 4800
+Wire Wire Line
+	5200 4600 5100 4600
+Wire Wire Line
+	5000 4450 5100 4450
+Wire Wire Line
+	5100 4450 5100 4600
+NoConn ~ 7100 5200
+NoConn ~ 7100 4700
+NoConn ~ 7100 5300
+NoConn ~ 7100 5400
+NoConn ~ 7100 5500
+NoConn ~ 7100 5800
+NoConn ~ 7100 5900
+NoConn ~ 7100 6000
+NoConn ~ 7100 6100
+$Comp
+L C C921
+U 1 1 5774E0E0
+P 5700 7100
+F 0 "C921" H 5750 7200 50  0000 L CNN
+F 1 "10uF" H 5750 7000 50  0000 L CNN
+F 2 "" H 5700 7100 60  0000 C CNN
+F 3 "" H 5700 7100 60  0000 C CNN
+	1    5700 7100
+	1    0    0    -1
+$EndComp
+Wire Wire Line
+	5700 7300 5700 7350
+Connection ~ 5700 7350
+Wire Wire Line
+	5700 6900 5700 6850
+Connection ~ 5700 6850
 $EndSCHEMATC

Commit message: = UPD: set values and manufacturer ref for components
Parts:
- C904: Manuf Ref (none) -> 0603X475K6R3CT; Manufacturer (none) -> Walsin
- L901: value INDUCTOR -> FB120; Manuf Ref (none) -> BLM18TG121TN1D; Manufacturer (none) -> Murata
- R905: Manuf Ref (none) -> CRCW06036K49FKEA; Manufacturer (none) -> Vishay
- R909, R910: Manuf Ref (none) -> CRCW0603330RFKEA; Manufacturer (none) -> Vishay
Changed lines of the file:
@@
 F 2 "" H 3200 2150 60  0000 C CNN
 F 3 "" H 3200 2150 60  0000 C CNN
+F 4 "Vishay" V 3200 2150 60  0001 C CNN "Manufacturer"
+F 5 "CRCW06036K49FKEA" V 3200 2150 60  0001 C CNN "Manuf Ref"
 	1    3200 2150
 	1    0    0    -1
@@
 F 2 "" H 3200 1250 60  0000 C CNN
 F 3 "" H 3200 1250 60  0000 C CNN
+F 4 "Walsin" H 3200 1250 60  0001 C CNN "Manufacturer"
+F 5 "0603X475K6R3CT" H 3200 1250 60  0001 C CNN "Manuf Ref"
 	1    3200 1250
 	1    0    0    -1
@@
 U 1 1 5641F57A
 P 2800 2700
-F 0 "L901" V 2750 2700 40  0000 C CNN
-F 1 "INDUCTOR" V 2900 2700 40  0000 C CNN
+F 0 "L901" V 2925 2700 50  0000 C CNN
+F 1 "FB120" V 2750 2700 40  0000 C CNN
 F 2 "" H 2800 2700 60  0000 C CNN
 F 3 "" H 2800 2700 60  0000 C CNN
+F 4 "Murata" V 2800 2700 60  0001 C CNN "Manufacturer"
+F 5 "BLM18TG121TN1D" V 2800 2700 60  0001 C CNN "Manuf Ref"
 	1    2800 2700
 	0    -1   -1   0
@@
 F 2 "" H 9800 2650 60  0000 C CNN
 F 3 "" H 9800 2650 60  0000 C CNN
+F 4 "Vishay" V 9800 2650 60  0001 C CNN "Manufacturer"
+F 5 "CRCW0603330RFKEA" V 9800 2650 60  0001 C CNN "Manuf Ref"
 	1    9800 2650
 	1    0    0    -1
@@
 F 2 "" H 10200 2650 60  0000 C CNN
 F 3 "" H 10200 2650 60  0000 C CNN
+F 4 "Vishay" V 10200 2650 60  0001 C CNN "Manufacturer"
+F 5 "CRCW0603330RFKEA" V 10200 2650 60  0001 C CNN "Manuf Ref"
 	1    10200 2650
 	-1   0    0    1
