File: pico-ice40-1k/hardware/prj_kicad/picow-1k-power.sch (KiCad schematic (older format))
At the start: 35 parts, among them P3 CONN_DC-2.0, U200 TPS560200, U201 LD6815, U202 TPS560200

Commit message: = UPD: Update hardware for rev 0.2.1 board (mainly bugfix)
Parts:
- added P200: CONN_FIX, symbol CONN_FIX
- added R205: 15k, symbol R
- added R206: 7,5k, symbol R
- added R207: 1k, symbol R
- added R208: R, symbol R
- added TP203, TP204, TP205, TP206, TP207: CONN_1, symbol CONN_1
- C224, C225, C226, C228: value C -> 100nF
- C227: value C -> 10uF
- L202: value INDUCTOR -> 10uH; Manuf Ref (none) -> TYS4012100M-10; Manufacturer (none) -> Laird Technologies
Connections:
- wire segments 97 -> 115
Other:
- moved on the sheet: C205, C224, C225, C226, C227

Commit message: = UPD: set values and manufacturer ref for components
Parts:
- C211: value 4,7uF -> 10uF; Manuf Ref (none) -> 0805X106K160CT; Manufacturer (none) -> Walsin
- C214, C215, C216: value C -> 100nF; Manuf Ref (none) -> C0603C104K4RACTU; Manufacturer (none) -> Kemet
- C224: Manuf Ref (none) -> C0603C104K4RACTU; Manufacturer (none) -> Kemet
- U201: Manuf Ref (none) -> LD6815TD/25P; Manufacturer (none) -> NXP
Changed lines of the file:
@@
 F 2 "" H 4150 6200 60  0000 C CNN
 F 3 "" H 4150 6200 60  0000 C CNN
+F 4 "NXP" H 4150 6200 60  0001 C CNN "Manufacturer"
+F 5 "LD6815TD/25P" H 4150 6200 60  0001 C CNN "Manuf Ref"
 	1    4150 6200
 	1    0    0    -1
@@
 P 4850 6350
 F 0 "C211" H 4900 6450 50  0000 L CNN
-F 1 "4,7uF" H 4900 6250 50  0000 L CNN
+F 1 "10uF" H 4900 6250 50  0000 L CNN
 F 2 "" H 4850 6350 60  0000 C CNN
 F 3 "" H 4850 6350 60  0000 C CNN
+F 4 "Walsin" H 4850 6350 60  0001 C CNN "Manufacturer"
+F 5 "0805X106K160CT" H 4850 6350 60  0001 C CNN "Manuf Ref"
 	1    4850 6350
 	1    0    0    -1
@@
 P 7150 4100
 F 0 "C214" H 7200 4200 50  0000 L CNN
-F 1 "C" H 7200 4000 50  0000 L CNN
+F 1 "100nF" H 7200 4000 50  0000 L CNN
 F 2 "" H 7150 4100 60  0000 C CNN
 F 3 "" H 7150 4100 60  0000 C CNN
+F 4 "Kemet" H 7150 4100 60  0001 C CNN "Manufacturer"
+F 5 "C0603C104K4RACTU" H 7150 4100 60  0001 C CNN "Manuf Ref"
 	1    7150 4100
 	1    0    0    -1
@@
 P 7450 4100
 F 0 "C215" H 7500 4200 50  0000 L CNN
-F 1 "C" H 7500 4000 50  0000 L CNN
+F 1 "100nF" H 7500 4000 50  0000 L CNN
 F 2 "" H 7450 4100 60  0000 C CNN
 F 3 "" H 7450 4100 60  0000 C CNN
+F 4 "Kemet" H 7450 4100 60  0001 C CNN "Manufacturer"
+F 5 "C0603C104K4RACTU" H 7450 4100 60  0001 C CNN "Manuf Ref"
 	1    7450 4100
 	1    0    0    -1
@@
 P 7750 4100
 F 0 "C216" H 7800 4200 50  0000 L CNN
-F 1 "C" H 7800 4000 50  0000 L CNN
+F 1 "100nF" H 7800 4000 50  0000 L CNN
 F 2 "" H 7750 4100 60  0000 C CNN
 F 3 "" H 7750 4100 60  0000 C CNN
+F 4 "Kemet" H 7750 4100 60  0001 C CNN "Manufacturer"
+F 5 "C0603C104K4RACTU" H 7750 4100 60  0001 C CNN "Manuf Ref"
 	1    7750 4100
 	1    0    0    -1
@@
 F 2 "" H 7750 2800 60  0000 C CNN
 F 3 "" H 7750 2800 60  0000 C CNN
+F 4 "Kemet" H 7750 2800 60  0001 C CNN "Manufacturer"
+F 5 "C0603C104K4RACTU" H 7750 2800 60  0001 C CNN "Manuf Ref"
 	1    7750 2800
 	1    0    0    -1
