File: pico-ice40-1k/hardware/prj_kicad/picow-1k.kicad_pcb (KiCad board)
At the start: 2 copper layers, 100 x 72 mm, 154 parts, among them P1 CONN_RJ45-L, P2 CONN_VGA, P3 CONN_DC-2.0, P4 CONN_12, P5 CONN_12, P6 CONN_2, Q901 BC846, SW1 SW_PUSH, SW2 SW_PUSH, SW3 SW_PUSH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

Commit message: = UPD: Update hardware for rev 0.2.1 board (mainly bugfix)
Parts:
- removed Pico-ITX_Holes: VAL**, Pico-ITX_Holes
- added C921: 10uF, SMD0805, F.Cu at (123.4, 104.5)
- added P200: CONN_FIX, Pico-ITX_Holes, F.Cu at (100.0, 50.0)
- added R205: 15k, SMD0603, F.Cu at (199.1, 65.4)
- added R206: 7,5k, SMD0603, F.Cu at (199.1, 67.9)
- added R207: 1k, SMD0603, F.Cu at (185.2, 75.2)
- added R208: R, SMD0603, F.Cu at (183.7, 75.2)
- added TP203: CONN_1, TP_PIN, F.Cu at (171.6, 106.3)
- added TP204: CONN_1, TP_PIN, F.Cu at (130.6, 74.1)
- added TP205: CONN_1, TP_PIN, F.Cu at (103.9, 77.4)
- added TP206: CONN_1, TP_PIN, F.Cu at (178.2, 120.5)
- added TP207: CONN_1, TP_SMD, B.Cu at (194.9, 67.3)
- C109: value 47uF -> 22uF
- C211: footprint SMD0603 -> SMD0805
- C224, C225, C226, C228: value C -> 100nF
- C227: value C -> 10uF; footprint C_TAJB -> SMD0805
- L101: value 4,7uH -> 10uH
- L202: value INDUCTOR -> 10uH
- R121, R123: value R -> 120
- R122: value R -> 60
- TP901, TP902: footprint TP_PIN -> TP_SMD; moved to B.Cu
- X1: value OSC -> 25MHz; footprint Q_TXC_5x3 -> Q_HC536
- moved C211 19.3 mm to (181.9, 76.8)
- moved R911 12.5 mm to (102.6, 66.1), turned to 0 degrees
- moved Q901 10.8 mm to (104.6, 64.6), turned to 270 degrees
- moved TP201 4.81 mm to (194.8, 71.3)
- moved C205 0.70 mm to (190.0, 73.1)
- moved C217 0.43 mm to (145.9, 71.7)
- moved TP902 0.38 mm to (116.6, 105.2)
- moved C203 0.20 mm to (193.2, 70.3)
- moved R201 0.15 mm to (191.7, 70.3)
- moved R202 0.15 mm to (190.1, 70.3)
- moved L200 0.15 mm to (196.3, 67.3)
- moved U200 0.15 mm to (192.2, 67.1)
- moved X900 0.15 mm to (104.6, 82.8)
- moved TP901 0.13 mm to (119.6, 105.2)
- moved X1 0.13 mm to (148.9, 71.5)
Connections:
- U200 pad 1: +Vin -> N-00000220
- U202 pad 1: +Vin -> N-00000219
- U900 pad 32: N-00000111 (its old number) -> GND
Routing:
- net GND: track 955.3 -> 1102.1 mm, vias 142 -> 151
- net +Vin: track 165.1 -> 141.5 mm
- net ETH_LED1: track 30.3 -> 43.3 mm
- net N-00000147: track 13.3 -> 4.30 mm
- net N-00000219: track 0.00 -> 8.62 mm, vias 0 -> 2
- net N-00000220: track 0.00 -> 7.12 mm, vias 0 -> 1
- net PLD_IT: track 46.3 -> 42.9 mm, vias 4 -> 2
- net LED2: track 30.3 -> 29.3 mm
- net LED1: track 30.7 -> 29.9 mm
- net LED3: track 29.9 -> 29.1 mm
- net LED4: track 30.9 -> 30.2 mm
- net N-00000151: track 1.83 -> 2.56 mm
- net LED0: track 31.2 -> 30.5 mm
- net N-00000107: track 2.82 -> 2.41 mm, vias 0 -> 1
- net N-00000106: track 5.80 -> 5.78 mm, vias 0 -> 1
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- added copper zone on F.Cu, net GND
Other:
- board text added: "0.2.1"
- board text added: "GND"

Commit message: = UPD: update silkscreen for components values
Parts:
- C106: value C -> 2,2uF
- C107, C214, C215, C216: value C -> 100nF
- C211: value 4,7uF -> 10uF
- L102: value FB100 -> FB120
- L103, L901: value INDUCTOR -> FB120
Changed lines of the file:
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@@
   )
   (setup
-    (last_trace_width 0.4064)
+    (last_trace_width 0.2032)
     (user_trace_width 0.1524)
     (user_trace_width 0.2032)
@@
       (effects (font (size 0.762 0.762) (thickness 0.1016)))
     )
-    (fp_text value INDUCTOR (at 0 0 180) (layer F.SilkS) hide
+    (fp_text value FB120 (at 0 0 180) (layer F.SilkS) hide
       (effects (font (size 0.20066 0.20066) (thickness 0.0508)))
     )
@@
       (effects (font (size 0.762 0.762) (thickness 0.1016)))
     )
-    (fp_text value C (at 0 0 180) (layer F.SilkS) hide
+    (fp_text value 2,2uF (at 0 0 180) (layer F.SilkS) hide
       (effects (font (size 0.20066 0.20066) (thickness 0.0508)))
     )
@@
       (effects (font (size 0.762 0.762) (thickness 0.1016)))
     )
-    (fp_text value C (at 0 0 270) (layer F.SilkS) hide
+    (fp_text value 100nF (at 0 0 270) (layer F.SilkS) hide
       (effects (font (size 0.20066 0.20066) (thickness 0.0508)))
     )
@@
       (effects (font (size 0.762 0.762) (thickness 0.1016)))
     )
-    (fp_text value C (at 0 0 180) (layer F.SilkS) hide
+    (fp_text value 100nF (at 0 0 180) (layer F.SilkS) hide
       (effects (font (size 0.20066 0.20066) (thickness 0.0508)))
     )
@@
       (effects (font (size 0.762 0.762) (thickness 0.1016)))
     )
-    (fp_text value C (at 0 0 180) (layer F.SilkS) hide
+    (fp_text value 100nF (at 0 0 180) (layer F.SilkS) hide
       (effects (font (size 0.20066 0.20066) (thickness 0.0508)))
     )
@@
       (effects (font (size 0.762 0.762) (thickness 0.1016)))
     )
-    (fp_text value C (at 0 0 270) (layer F.SilkS) hide
+    (fp_text value 100nF (at 0 0 270) (layer F.SilkS) hide
       (effects (font (size 0.20066 0.20066) (thickness 0.0508)))
     )
@@
       (effects (font (size 0.762 0.762) (thickness 0.1016)))
     )
-    (fp_text value FB100 (at 0 0 90) (layer F.SilkS) hide
+    (fp_text value FB120 (at 0 0 90) (layer F.SilkS) hide
       (effects (font (size 0.20066 0.20066) (thickness 0.0508)))
     )
@@
       (effects (font (size 0.762 0.762) (thickness 0.1016)))
     )
-    (fp_text value INDUCTOR (at 0 0 90) (layer F.SilkS) hide
+    (fp_text value FB120 (at 0 0 90) (layer F.SilkS) hide
       (effects (font (size 0.20066 0.20066) (thickness 0.0508)))
     )
@@
       (effects (font (size 0.762 0.762) (thickness 0.1016)))
     )
-    (fp_text value 4,7uF (at 0 0 180) (layer F.SilkS) hide
+    (fp_text value 10uF (at 0 0 180) (layer F.SilkS) hide
       (effects (font (size 0.2 0.2) (thickness 0.05)))
     )
